File: Hardware/Qwiic_Spectral_Sensor-AS726x.brd (EAGLE design)
At the start: 25.4 x 25.4 mm, 32 parts, among them J1 Qwiic Right Angle, J2 Serial Interface, J4 Qwiic Right Angle, J5 Flash Programming, U1 IR, U3 4MB Flash

Commit message: Continued to update with checklist
Parts:
- moved D4 0.13 mm to (22.2, 17.4)
Routing:
- net 3.3V: track 88.3 -> 91.4 mm
Other:
- board text added: "Opt. LED"
