File: Hardware/Qwiic_Spectral_Sensor-AS726x.brd (EAGLE design)
At the start: 25.4 x 25.4 mm, 32 parts, among them J1 Qwiic Right Angle, J2 Serial Interface, J4 Qwiic Right Angle, J5 Flash Programming, U1 IR, U3 4MB Flash

Commit message: Changed version number
Other:
- board text added: "V10"
- board text removed: "V01"
Changed lines of the file:
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@@
 <text x="3.683" y="17.78" size="1.016" layer="21" font="vector" ratio="15" align="center">Spectral
 Sensor</text>
-<text x="3.429" y="0.762" size="1.016" layer="16" ratio="20" rot="MR0" align="bottom-center">V01</text>
+<text x="3.429" y="0.762" size="1.016" layer="16" ratio="20" rot="MR0" align="bottom-center">V10</text>
 <text x="5.334" y="11.43" size="0.889" layer="22" ratio="15" rot="MR90" align="bottom-center">JP2</text>
 <text x="16.51" y="-21.59" size="1.778" layer="51">Nathan Seidle</text>
